File: PCB Design/ece196-project-sketch.kicad_sch (KiCad schematic)
At the start: 41 parts, among them J1 USB_C_Receptacle

Commit message: Add files via upload
Parts:
- removed MOS_BST1: RUF025N02TL, RUF025N02TL, symbol SamacSys_Symbols:RUF025N02TL
- added Q1: 2N7000, Package_TO_SOT_THT:TO-92_Inline, symbol Transistor_FET:2N7000
Connections:
- net +BATT: now also Q1.3 (D)
- net BOOST_TRIG: now also Q1.2 (G)
- net at C_BST1.1, IC_BST1.5 (VIN), L_BST1.1: now also Q1.1 (S)
Changed lines of the file:
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@@
+    (stroke (width 0) (type default))
+  )
+  (wire (pts (xy 157.48 27.94) (xy 162.56 27.94))
     (stroke (width 0) (type default))
   )
@@
         (path "/8857b4b0-9906-42ef-aa31-1981db0a7282"
           (reference "#PWR01") (unit 1)
-        )
-      )
-    )
-  )
-  (symbol (lib_id "SamacSys_Symbols:RUF025N02TL") (at 167.64 35.56 90) (unit 1)
-    (in_bom yes) (on_board yes) (dnp no) (fields_autoplaced)
-    (property "Reference" "MOS_BST1" (at 165.1 21.59 90)
-      (effects (font (size 1.27 1.27)))
-    )
-    (property "Value" "RUF025N02TL" (at 165.1 24.13 90)
-      (effects (font (size 1.27 1.27)))
-    )
-    (property "Footprint" "RUF025N02TL" (at 266.37 24.13 0)
-      (effects (font (size 1.27 1.27)) (justify left top) hide)
-    )
-    (property "Datasheet" "https://fscdn.rohm.com/en/products/databook/datasheet/discrete/transistor/mosfet/ruf025n02tl-e.pdf" (at 366.37 24.13 0)
-      (effects (font (size 1.27 1.27)) (justify left top) hide)
-    )
-    (property "Height" "0.85" (at 566.37 24.13 0)
-      (effects (font (size 1.27 1.27)) (justify left top) hide)
-    )
-    (property "Mouser Part Number" "755-RUF025N02TL" (at 666.37 24.13 0)
-      (effects (font (size 1.27 1.27)) (justify left top) hide)
-    )
-    (property "Mouser Price/Stock" "https://www.mouser.co.uk/ProductDetail/ROHM-Semiconductor/RUF025N02TL?qs=IJ4m%2FCjbxWeiXw%2F4C8Ss6Q%3D%3D" (at 766.37 24.13 0)
-      (effects (font (size 1.27 1.27)) (justify left top) hide)
-    )
-    (property "Manufacturer_Name" "ROHM Semiconductor" (at 866.37 24.13 0)
-      (effects (font (size 1.27 1.27)) (justify left top) hide)
-    )
-    (property "Manufacturer_Part_Number" "RUF025N02TL" (at 966.37 24.13 0)
-      (effects (font (size 1.27 1.27)) (justify left top) hide)
-    )
-    (pin "1")
-    (pin "2")
-    (pin "3")
-    (instances
-      (project "ece196-project-sketch"
-        (path "/8857b4b0-9906-42ef-aa31-1981db0a7282"
-          (reference "MOS_BST1") (unit 1)
         )
       )
@@
         )
       )
+    )
+  )
+  (symbol (lib_id "Transistor_FET:2N7000") (at 167.64 30.48 90) (unit 1)
+    (in_bom yes) (on_board yes) (dnp no) (fields_autoplaced)
+    (property "Reference" "Q1" (at 167.64 21.59 90)
+      (effects (font (size 1.27 1.27)))
+    )
+    (property "Value" "2N7000" (at 167.64 24.13 90)
+      (effects (font (size 1.27 1.27)))
+    )
+    (property "Footprint" "Package_TO_SOT_THT:TO-92_Inline" (at 169.545 25.4 0)
+      (effects (font (size 1.27 1.27) italic) (justify left) hide)
+    )
+    (property "Datasheet" "https://www.vishay.com/docs/70226/70226.pdf" (at 167.64 30.48 0)
+      (effects (font (size 1.27 1.27)) (justify left) hide)
+    )
+    (pin "1")
+    (pin "2")
+    (pin "3")
+    (instances
+      (project "ece196-project-sketch"
+        (path "/8857b4b0-9906-42ef-aa31-1981db0a7282"
+          (reference "Q1") (unit 1)
+        )
+      )
